File: doc/eagle/uno_shield/main.sch (EAGLE design)
At the start: 15 parts, among them U1 ARDUINOR3-BPLACE

Commit message: [ add ] routed board, main.png
Parts:
- removed R2, R4: 1k, rcl:R-EU_0204/5
- removed R3: (no value), rcl:R-TRIMM64X
- added R8: (no value), resistor:R-TRIMM3339P
- R1: device rcl:R-TRIMM64X -> resistor:R-TRIMM3339P
Connections:
- removed net N$1: R1.E, R2.1
- removed net N$2: R3.E, R4.1
- net ADC_VCAP: now also R8.S; no longer R1.S
- net ADC_VOUT: now also R1.S; no longer R3.S
- net BUT_MINUS: now also S4.1, S4.2, U1.A5/SCL; no longer S2.1, S2.2, U1.A3
- net BUT_MODE: now also S2.1, S2.2, U1.A3; no longer S1.1, S1.2, U1.A4/SDA
- net BUT_PLUS: now also S1.1, S1.2, U1.A4/SDA; no longer S3.1, S3.2, U1.A2
- net BUT_SAVE: now also S3.1, S3.2, U1.A2; no longer S4.1, S4.2, U1.A5/SCL
- net GND: now also R1.A, R8.A; no longer R2.2, R4.2
- net LCD_EN: now also U1.D6; no longer U1.D7
- net LCD_RS: now also U1.D7; no longer U1.D6
- net UNO_5V: now also R1.E, R8.E; no longer R1.A, R3.A
Other:
- moved on the sheet: R1, R7
