File: doc/eagle/voltage_scaling_stage/main.sch (EAGLE design)
At the start: 6 parts, among them U1 AD8278ARMZ

Commit message: [ update ] eagle/voltage_scaling_stage
Parts:
- removed R6: 1M, rcl:R-EU_0204/5
- R2, R4: value 40k -> 50k
Connections:
- removed net N$4: U1.REF
- removed net VIN_DIFF: R6.1, U1.OUT
- net GND: now also U1.REF, U1.SENSE
- net VIN_MINUS_DIV: no longer R6.2
Other:
- note added: "gain = 1"
- note removed: "gain = r6 / r3 = 1"
Changed lines of the file:
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@@
 <part name="U1" library="ADI-AD8278ARMZ" deviceset="AD8278ARMZ" device=""/>
 <part name="R1" library="rcl" deviceset="R-EU_" device="0204/5" value="1M"/>
-<part name="R2" library="rcl" deviceset="R-EU_" device="0204/5" value="40k"/>
+<part name="R2" library="rcl" deviceset="R-EU_" device="0204/5" value="50k"/>
 <part name="R3" library="rcl" deviceset="R-EU_" device="0204/5" value="1M"/>
-<part name="R4" library="rcl" deviceset="R-EU_" device="0204/5" value="40k"/>
-<part name="R6" library="rcl" deviceset="R-EU_" device="0204/5" value="1M"/>
+<part name="R4" library="rcl" deviceset="R-EU_" device="0204/5" value="50k"/>
 </parts>
 <sheets>
 <sheet>
 <plain>
-<text x="22.86" y="66.04" size="1.778" layer="91">gain = r6 / r3 = 1</text>
+<text x="20.32" y="53.34" size="1.778" layer="91">gain = 1</text>
 </plain>
 <instances>
@@
 <instance part="R3" gate="G$1" x="-15.24" y="63.5"/>
 <instance part="R4" gate="G$1" x="0" y="63.5"/>
-<instance part="R6" gate="G$1" x="20.32" y="43.18"/>
 </instances>
 <busses>
@@
 </segment>
 <segment>
-<pinref part="R6" gate="G$1" pin="2"/>
-<wire x1="25.4" y1="43.18" x2="27.94" y2="43.18" width="0.1524" layer="91"/>
-<label x="27.94" y="43.18" size="1.778" layer="95"/>
+<wire x1="10.16" y1="48.26" x2="20.32" y2="48.26" width="0.1524" layer="91"/>
+<label x="10.16" y="48.26" size="1.778" layer="95"/>
 </segment>
 </net>
@@
 <wire x1="-25.4" y1="22.86" x2="-48.26" y2="22.86" width="0.1524" layer="91"/>
 <label x="-48.26" y="22.86" size="1.778" layer="95"/>
+</segment>
+<segment>
+<pinref part="U1" gate="A" pin="REF"/>
+<wire x1="-25.4" y1="35.56" x2="-48.26" y2="35.56" width="0.1524" layer="91"/>
+<label x="-48.26" y="35.56" size="1.778" layer="95"/>
+</segment>
+<segment>
+<pinref part="U1" gate="A" pin="SENSE"/>
+<wire x1="-25.4" y1="33.02" x2="-48.26" y2="33.02" width="0.1524" layer="91"/>
+<label x="-48.26" y="33.02" size="1.778" layer="95"/>
 </segment>
 </net>
@@
 </segment>
 </net>
-<net name="VIN_DIFF" class="0">
-<segment>
-<pinref part="U1" gate="A" pin="OUT"/>
-<wire x1="10.16" y1="48.26" x2="12.7" y2="48.26" width="0.1524" layer="91"/>
-<wire x1="12.7" y1="48.26" x2="12.7" y2="53.34" width="0.1524" layer="91"/>
-<junction x="12.7" y="48.26"/>
-<wire x1="12.7" y1="53.34" x2="27.94" y2="53.34" width="0.1524" layer="91"/>
-<label x="27.94" y="53.34" size="1.778" layer="95"/>
-<wire x1="12.7" y1="48.26" x2="12.7" y2="43.18" width="0.1524" layer="91"/>
-<wire x1="12.7" y1="43.18" x2="15.24" y2="43.18" width="0.1524" layer="91"/>
-<pinref part="R6" gate="G$1" pin="1"/>
-</segment>
-</net>
 <net name="5V" class="0">
 <segment>
@@
 </segment>
 </net>
-<net name="N$4" class="0">
-<segment>
-<pinref part="U1" gate="A" pin="REF"/>
-<wire x1="-25.4" y1="35.56" x2="-48.26" y2="35.56" width="0.1524" layer="91"/>
-</segment>
-</net>

Commit message: [ update ] voltage_scaling_stage
Parts:
- added R5, R6: 51k, resistor:R-US_R1206
- added R7, R8: 1M, resistor:R-US_R1206
- added U2: AD8276ARZ, ADI-AD8276ARZ:AD8276ARZ
- R1, R3: value 1M -> 51k; device rcl:R-EU_0204/5 -> resistor:R-US_R1206
- R2, R4: value 50k -> 1M; device rcl:R-EU_0204/5 -> resistor:R-US_R1206
- U1: value AD8278ARMZ -> AD8276ARZ; device ADI-AD8278ARMZ:AD8278ARMZ -> ADI-AD8276ARZ:AD8276ARZ
Connections:
- removed net VIN_MINUS: R1.1
- removed net VIN_MINUS_DIV: R1.2, R2.1, U1.-IN
- removed net VIN_PLUS: R3.1
- removed net VIN_PLUS_DIV: R3.2, R4.1, U1.+IN
- new net VCAP_DIFF: U2.OUT, U2.SENSE
- new net VCAP_MINUS_DIV: R1.1, R2.2, U2.-IN
- new net VCAP_PLUS_DIV: R3.1, R4.2, U2.+IN
- new net VOUT_DIFF: U1.OUT, U1.SENSE
- new net VOUT_MINUS: R7.1
- new net VOUT_MINUS_DIV: R5.1, R7.2, U1.-IN
- new net VOUT_PLUS: R8.1
- new net VOUT_PLUS_DIV: R6.1, R8.2, U1.+IN
- net 5V: now also U2.+VS
- net GND: now also R1.2, R3.2, R5.2, R6.2, U2.-VS, U2.REF; no longer R2.2, R4.2, U1.SENSE
Other:
- note added: "/21 voltage dividor"
- note added: "gain = 1. DS figure 38, page 13"
- note removed: "gain = 1"
- moved on the sheet: U1
